File: hardware/electronics/spike_n_hold/spike_n_hold/spike_n_hold.kicad_pcb (KiCad board)
At the start: 2 copper layers, 132 parts, among them J1 input_trigger_2, J10 input_trigger_6, J11 input_trigger_5, J12 to_solenoid_6, J13 to_solenoid_5, J2 input_trigger_1, J3 to_solenoid_2, J4 to_solenoid_1, J5 input_trigger_4, J6 input_trigger_3, J7 to_solenoid_4, J8 to_solenoid_3, J9 Barrel_Jack_MountingPin, Q1 MJH11021G, Q10 MJH11021G, Q11 MPSA42, Q12 MPSA42, Q13 MPSA42, Q14 MPSA42, Q15 MJH11022G, Q16 MJH11022G, Q17 MJH11021G, Q18 MJH11021G, Q19 MPSA42, Q2 MJH11021G, Q20 MPSA42, Q21 MPSA42, Q22 MPSA42, Q23 MJH11022G, Q24 MJH11022G, Q3 MPSA42, Q4 MPSA42, Q5 MPSA42, Q6 MPSA42, Q7 MJH11022G, Q8 MJH11022G, Q9 MJH11021G, U1 LM555xM, U2 LM555xM, U3 LM555xM, U4 LM555xM, U5 LM2596T-12, U6 LM555xM, U7 LM555xM

Commit message: reimplementation, 2 modules per board, as they are equivalent to one odour channel, or one dilution step
Parts:
- removed C10, C17, C18, C9: 10nF, Capacitor_THT:C_Disc_D5.1mm_W3.2mm_P5.00mm
- removed C12, C13, C19, C20: 10µF, Capacitor_THT:C_Disc_D5.1mm_W3.2mm_P5.00mm
- removed C14, C16, C7, C8: 680pF, Capacitor_THT:C_Disc_D5.1mm_W3.2mm_P5.00mm
- removed D10, D11, D12, D13, D14, D18, D19, D20, D21, D22, D23, D9: 1N4005, Diode_THT:D_DO-41_SOD81_P10.16mm_Horizontal
- removed D15, D16, D24, D25: 1N47xxA, Diode_THT:D_DO-41_SOD81_P10.16mm_Horizontal
- removed J10: input_trigger_6, Connector_PinHeader_2.54mm:PinHeader_1x02_P2.54mm_Vertical
- removed J11: input_trigger_5, Connector_PinHeader_2.54mm:PinHeader_1x02_P2.54mm_Vertical
- removed J12: to_solenoid_6, Connector_PinHeader_2.54mm:PinHeader_1x02_P2.54mm_Vertical
- removed J13: to_solenoid_5, Connector_PinHeader_2.54mm:PinHeader_1x02_P2.54mm_Vertical
- removed J5: input_trigger_4, Connector_PinHeader_2.54mm:PinHeader_1x02_P2.54mm_Vertical
- removed J6: input_trigger_3, Connector_PinHeader_2.54mm:PinHeader_1x02_P2.54mm_Vertical
- removed J7: to_solenoid_4, Connector_PinHeader_2.54mm:PinHeader_1x02_P2.54mm_Vertical
- removed J8: to_solenoid_3, Connector_PinHeader_2.54mm:PinHeader_1x02_P2.54mm_Vertical
- removed Q10, Q17, Q18, Q9: MJH11021G, Package_TO_SOT_THT:TO-247-3_Vertical
- removed Q11, Q12, Q13, Q14, Q19, Q20, Q21, Q22: MPSA42, Package_TO_SOT_THT:TO-92L_Inline_Wide
- removed Q15, Q16, Q23, Q24: MJH11022G, Package_TO_SOT_THT:TO-247-3_Vertical
- removed R15, R17, R22, R24, R29, R30, R37, R38: 10k, Resistor_THT:R_Axial_DIN0411_L9.9mm_D3.6mm_P12.70mm_Horizontal
- removed R16, R18, R31, R32: 4.7k, Resistor_THT:R_Axial_DIN0411_L9.9mm_D3.6mm_P12.70mm_Horizontal
- removed R19, R20, R21, R23, R25, R26, R33, R34, R35, R36, R39, R40: 330, Resistor_THT:R_Axial_DIN0411_L9.9mm_D3.6mm_P12.70mm_Horizontal
- removed R27, R28, R41, R42: 2k, Resistor_THT:R_Axial_DIN0411_L9.9mm_D3.6mm_P12.70mm_Horizontal
- removed U3, U4, U6, U7: LM555xM, Package_DIP:DIP-8_W7.62mm_LongPads
- moved C15 90.8 mm to (191.0, 118.0), turned to 180 degrees
- moved L1 77.7 mm to (187.0, 106.5), turned to 0 degrees
- moved U5 69.8 mm to (188.5, 91.5), turned to 270 degrees
- moved J9 67.1 mm to (189.0, 81.5), turned to 270 degrees
- moved D17 62.0 mm to (179.0, 98.5), turned to 270 degrees
- moved C11 58.2 mm to (180.5, 89.5), turned to 180 degrees
Routing:
- net +12V: track 328.4 -> 172.6 mm
- net +24V: track 181.1 -> 47.6 mm, vias 6 -> 0
- net Net-(D16-Pad1): track 58.6 -> 0.00 mm
- net Net-(D15-Pad1): track 53.6 -> 0.00 mm
- net Net-(D12-Pad1): track 43.7 -> 0.00 mm
- net Net-(D11-Pad1): track 38.4 -> 0.00 mm
- net Net-(Q14-Pad3): track 20.3 -> 0.00 mm
- net input_trigger4: track 19.1 -> 0.00 mm
- net input_trigger3: track 17.6 -> 0.00 mm
- net Net-(C13-Pad1): track 17.5 -> 0.00 mm
- net Net-(Q13-Pad3): track 17.3 -> 0.00 mm
- net Net-(D10-Pad1): track 15.7 -> 0.00 mm
- net Net-(C12-Pad1): track 15.6 -> 0.00 mm
- net Net-(D13-Pad1): track 14.8 -> 0.00 mm
- net Net-(Q12-Pad3): track 14.6 -> 0.00 mm
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