File: hardware/electronics/spike_n_hold/spike_n_hold/spike_n_hold.sch (KiCad schematic (older format))
At the start: 27 parts

Commit message: fix capacitor value
Parts:
- C5: renamed from C?; value 680µF -> 220µF
- gave numbers to parts that had none: 26
Other:
- note added: "C2 and R1 values should/can be changed to\nincrease/decrease the duration of the spike period"
Changed lines of the file:
@@
 $EndDescr
 $Comp
-L Device:R_Small R?
+L Device:R_Small R6
 U 1 1 5FD8C64E
 P 1650 4950
-F 0 "R?" H 1591 4904 50  0000 R CNN
+F 0 "R6" H 1591 4904 50  0000 R CNN
 F 1 "330" H 1591 4995 50  0000 R CNN
 F 2 "" H 1650 4950 50  0001 C CNN
@@
 $EndComp
 $Comp
-L power:GND #PWR?
+L power:GND #PWR09
 U 1 1 5FD91FD0
 P 2550 7100
-F 0 "#PWR?" H 2550 6850 50  0001 C CNN
+F 0 "#PWR09" H 2550 6850 50  0001 C CNN
 F 1 "GND" V 2555 6972 50  0000 R CNN
 F 2 "" H 2550 7100 50  0001 C CNN
@@
 	2550 7100 2550 7050
 $Comp
-L Connector:Screw_Terminal_01x02 J?
+L Connector:Screw_Terminal_01x02 J3
 U 1 1 5FD93E5A
 P 3750 5700
-F 0 "J?" V 3622 5780 50  0000 L CNN
+F 0 "J3" V 3622 5780 50  0000 L CNN
 F 1 "to_solenoid" V 3713 5780 50  0000 L CNN
 F 2 "" H 3750 5700 50  0001 C CNN
@@
 $EndComp
 $Comp
-L Diode:1N47xxA D?
+L Diode:1N47xxA D5
 U 1 1 5FD94D24
 P 2550 6150
-F 0 "D?" H 2550 6367 50  0000 C CNN
+F 0 "D5" H 2550 6367 50  0000 C CNN
 F 1 "1N47xxA" H 2550 6276 50  0000 C CNN
 F 2 "Diode_THT:D_DO-41_SOD81_P10.16mm_Horizontal" H 2550 5975 50  0001 C CNN
@@
 $EndComp
 $Comp
-L Diode:1N4005 D?
+L Diode:1N4005 D4
 U 1 1 5FD992D4
 P 2550 5700
-F 0 "D?" H 2550 5483 50  0000 C CNN
+F 0 "D4" H 2550 5483 50  0000 C CNN
 F 1 "1N4005" H 2550 5574 50  0000 C CNN
 F 2 "Diode_THT:D_DO-41_SOD81_P10.16mm_Horizontal" H 2550 5525 50  0001 C CNN
@@
 	2550 6000 2550 5850
 $Comp
-L Diode:1N4005 D?
+L Diode:1N4005 D3
 U 1 1 5FD9B1F7
 P 3200 5250
-F 0 "D?" V 3246 5170 50  0000 R CNN
+F 0 "D3" V 3246 5170 50  0000 R CNN
 F 1 "1N4005" V 3155 5170 50  0000 R CNN
 F 2 "Diode_THT:D_DO-41_SOD81_P10.16mm_Horizontal" H 3200 5075 50  0001 C CNN
@@
 $EndComp
 $Comp
-L power:+12V #PWR?
+L power:+12V #PWR07
 U 1 1 5FFF83E5
 P 3200 5050
-F 0 "#PWR?" H 3200 4900 50  0001 C CNN
+F 0 "#PWR07" H 3200 4900 50  0001 C CNN
 F 1 "+12V" V 3215 5178 50  0000 L CNN
 F 2 "" H 3200 5050 50  0001 C CNN
@@
 	3500 5800 3500 6450
 $Comp
-L Device:R_Small R?
+L Device:R_Small R7
 U 1 1 600211A6
 P 1850 5950
-F 0 "R?" H 1791 5904 50  0000 R CNN
+F 0 "R7" H 1791 5904 50  0000 R CNN
 F 1 "330" H 1791 5995 50  0000 R CNN
 F 2 "" H 1850 5950 50  0001 C CNN
@@
 $EndComp
 $Comp
-L dk_Transistors-Bipolar-BJT-Single:MPSA42 Q?
+L dk_Transistors-Bipolar-BJT-Single:MPSA42 Q3
 U 1 1 60024F50
 P 2100 6350
-F 0 "Q?" H 2288 6403 60  0000 L CNN
+F 0 "Q3" H 2288 6403 60  0000 L CNN
 F 1 "MPSA42" H 2288 6297 60  0000 L CNN
 F 2 "digikey-footprints:TO-92-3" H 2300 6550 60  0001 L CNN
@@
 $EndComp
 $Comp
-L Device:R_Small R?
+L Device:R_Small R4
 U 1 1 6002F3C0
 P 2800 3700
-F 0 "R?" H 2741 3654 50  0000 R CNN
+F 0 "R4" H 2741 3654 50  0000 R CNN
 F 1 "10k" H 2741 3745 50  0000 R CNN
 F 2 "" H 2800 3700 50  0001 C CNN
@@
 $EndComp
 $Comp
-L Device:R_Small R?
+L Device:R_Small R5
 U 1 1 60033420
 P 2400 4250
-F 0 "R?" H 2341 4204 50  0000 R CNN
+F 0 "R5" H 2341 4204 50  0000 R CNN
 F 1 "4.7k" H 2341 4295 50  0000 R CNN
 F 2 "" H 2400 4250 50  0001 C CNN
@@
 $EndComp
 $Comp
-L Device:Q_NPN_Darlington_BCE Q?
+L Device:Q_NPN_Darlington_BCE Q4
 U 1 1 6003A207
 P 2450 6800
-F 0 "Q?" H 2640 6846 50  0000 L CNN
+F 0 "Q4" H 2640 6846 50  0000 L CNN
 F 1 "MJH11022G" H 2640 6755 50  0000 L CNN
 F 2 "" H 2650 6900 50  0001 C CNN
@@
 $EndComp
 $Comp
-L Device:Q_PNP_Darlington_BCE Q?
+L Device:Q_PNP_Darlington_BCE Q2
 U 1 1 6003EB44
 P 2800 4250
-F 0 "Q?" H 2990 4296 50  0000 L CNN
+F 0 "Q2" H 2990 4296 50  0000 L CNN
 F 1 "MJH11021G" H 2990 4205 50  0000 L CNN
 F 2 "" H 3000 4350 50  0001 C CNN
@@
 	2900 3550 2900 3700
 $Comp
-L power:+24V #PWR?
+L power:+24V #PWR04
 U 1 1 6002D4F0
 P 2900 3550
-F 0 "#PWR?" H 2900 3400 50  0001 C CNN
+F 0 "#PWR04" H 2900 3400 50  0001 C CNN
 F 1 "+24V" H 2915 3723 50  0000 C CNN
 F 2 "" H 2900 3550 50  0001 C CNN
@@
 	4050 2150 3800 2150
 $Comp
-L pspice:CAP C?
+L pspice:CAP C3
 U 1 1 5FD88E6E
 P 4050 2800
-F 0 "C?" V 4365 2800 50  0000 C CNN
+F 0 "C3" V 4365 2800 50  0000 C CNN
 F 1 "10nF" V 4274 2800 50  0000 C CNN
 F 2 "" H 4050 2800 50  0001 C CNN
@@
 	5450 3000 5450 3050
 $Comp
-L power:GND #PWR?
+L power:GND #PWR03
 U 1 1 5FD882A9
 P 5450 3150
-F 0 "#PWR?" H 5450 2900 50  0001 C CNN
+F 0 "#PWR03" H 5450 2900 50  0001 C CNN
 F 1 "GND" H 5455 2977 50  0000 C CNN
 F 2 "" H 5450 3150 50  0001 C CNN
@@
 	5450 2350 5450 2500
 $Comp
-L pspice:CAP C?
+L pspice:CAP C2
 U 1 1 5FD875CF
 P 5450 2750
-F 0 "C?" H 5272 2704 50  0000 R CNN
+F 0 "C2" H 5272 2704 50  0000 R CNN
 F 1 "10µF" H 5272 2795 50  0000 R CNN
 F 2 "" H 5450 2750 50  0001 C CNN
@@
 	4550 1450 4700 1450
 $Comp
-L Device:R_Small R?
+L Device:R_Small R1
 U 1 1 5FD85CF8
 P 4900 1500
-F 0 "R?" V 5096 1500 50  0000 C CNN
+F 0 "R1" V 5096 1500 50  0000 C CNN
 F 1 "2k" V 5005 1500 50  0000 C CNN
 F 2 "" H 4900 1500 50  0001 C CNN
@@
 	3350 2050 3350 1950
 $Comp
-L Device:R_Small R?
+L Device:R_Small R2
 U 1 1 5FD834A0
 P 3650 1850
-F 0 "R?" H 3591 1804 50  0000 R CNN
+F 0 "R2" H 3591 1804 50  0000 R CNN
 F 1 "10k" H 3591 1895 50  0000 R CNN
 F 2 "" H 3650 1850 50  0001 C CNN
@@
 	4500 1300 4550 1300
 $Comp
-L power:VCC #PWR?
+L power:VCC #PWR01
 U 1 1 5FD82952
 P 4500 1300
-F 0 "#PWR?" H 4500 1150 50  0001 C CNN
+F 0 "#PWR01" H 4500 1150 50  0001 C CNN
 F 1 "VCC" H 4515 1473 50  0000 C CNN
 F 2 "" H 4500 1300 50  0001 C CNN
@@
 	2850 2250 3050 2250
 $Comp
-L Transistor_BJT:MPSA42 Q?
+L Transistor_BJT:MPSA42 Q1
 U 1 1 5FD7F192
 P 3250 2250
-F 0 "Q?" H 3441 2296 50  0000 L CNN
+F 0 "Q1" H 3441 2296 50  0000 L CNN
 F 1 "MPSA42" H 3441 2205 50  0000 L CNN
 F 2 "Package_TO_SOT_THT:TO-92_Inline" H 3450 2175 50  0001 L CIN
@@
 	1400 2500 1800 2500
 $Comp
-L Diode:1N4005 D?
+L Diode:1N4005 D1
 U 1 1 5FD7DBAD
 P 2850 2400
-F 0 "D?" V 2804 2480 50  0000 L CNN
+F 0 "D1" V 2804 2480 50  0000 L CNN
 F 1 "1N4005" V 2895 2480 50  0000 L CNN
 F 2 "Diode_THT:D_DO-41_SOD81_P10.16mm_Horizontal" H 2850 2225 50  0001 C CNN
@@
 $EndComp
 $Comp
-L Device:R_Small R?
+L Device:R_Small R3
 U 1 1 5FD7D15C
 P 2550 2250
-F 0 "R?" V 2354 2250 50  0000 C CNN
+F 0 "R3" V 2354 2250 50  0000 C CNN
 F 1 "330" V 2445 2250 50  0000 C CNN
 F 2 "" H 2550 2250 50  0001 C CNN
@@
 	1400 2450 1400 2500
 $Comp
-L power:GND #PWR?
+L power:GND #PWR02
 U 1 1 5FD7C260
 P 1400 2600
-F 0 "#PWR?" H 1400 2350 50  0001 C CNN
+F 0 "#PWR02" H 1400 2350 50  0001 C CNN
 F 1 "GND" H 1405 2427 50  0000 C CNN
 F 2 "" H 1400 2600 50  0001 C CNN
@@
 $EndComp
 $Comp
-L Connector:Conn_Coaxial J?
+L Connector:Conn_Coaxial J1
 U 1 1 5FD7BC13
 P 1400 2250
-F 0 "J?" H 1328 2488 50  0000 C CNN
+F 0 "J1" H 1328 2488 50  0000 C CNN
 F 1 "Conn_Coaxial" H 1328 2397 50  0000 C CNN
 F 2 "" H 1400 2250 50  0001 C CNN
@@
 $EndComp
 $Comp
-L Timer:LM555xM U?
+L Timer:LM555xM U1
 U 1 1 5FD78A96
 P 4550 2150
-F 0 "U?" H 4550 2731 50  0000 C CNN
+F 0 "U1" H 4550 2731 50  0000 C CNN
 F 1 "LM555xM" H 4550 2640 50  0000 C CNN
 F 2 "Package_SO:SOIC-8_3.9x4.9mm_P1.27mm" H 5400 1750 50  0001 C CNN
@@
 Connection ~ 2300 4250
 $Comp
-L power:+24V #PWR?
+L power:+24V #PWR05
 U 1 1 6015360F
 P 5800 4200
-F 0 "#PWR?" H 5800 4050 50  0001 C CNN
+F 0 "#PWR05" H 5800 4050 50  0001 C CNN
 F 1 "+24V" H 5815 4373 50  0000 C CNN
 F 2 "" H 5800 4200 50  0001 C CNN
@@
 	6150 4500 6300 4500
 $Comp
-L power:GND #PWR?
+L power:GND #PWR08
 U 1 1 60157381
 P 6450 5050
-F 0 "#PWR?" H 6450 4800 50  0001 C CNN
+F 0 "#PWR08" H 6450 4800 50  0001 C CNN
 F 1 "GND" H 6455 4877 50  0000 C CNN
 F 2 "" H 6450 5050 50  0001 C CNN
@@
 Connection ~ 6450 5050
 $Comp
-L pspice:CAP C?
+L pspice:CAP C1
 U 1 1 5FD7C907
 P 2000 2250
-F 0 "C?" V 1685 2250 50  0000 C CNN
+F 0 "C1" V 1685 2250 50  0000 C CNN
 F 1 "680pF" V 1776 2250 50  0000 C CNN
 F 2 "" H 2000 2250 50  0001 C CNN
@@
 Connection ~ 6300 5050
 $Comp
-L Regulator_Switching:LM2596T-12 U?
+L Regulator_Switching:LM2596T-12 U2
 U 1 1 6016A039
 P 6800 4600
-F 0 "U?" H 6800 4967 50  0000 C CNN
+F 0 "U2" H 6800 4967 50  0000 C CNN
 F 1 "LM2596T-12" H 6800 4876 50  0000 C CNN
 F 2 "Package_TO_SOT_THT:TO-220-5_P3.4x3.7mm_StaggerOdd_Lead3.8mm_Vertical" H 6850 4350 50  0001 L CIN
@@
 $EndComp
 $Comp
-L Diode:1N5820 D?
+L Diode:1N5820 D2
 U 1 1 6016F0ED
 P 7500 4850
-F 0 "D?" V 7454 4930 50  0000 L CNN
+F 0 "D2" V 7454 4930 50  0000 L CNN
 F 1 "1N5820" V 7545 4930 50  0000 L CNN
 F 2 "Diode_THT:D_DO-201AD_P15.24mm_Horizontal" H 7500 4675 50  0001 C CNN
@@
 $EndComp
 $Comp
-L Device:L L?
+L Device:L L1
 U 1 1 6016FEA8
 P 8050 4700
-F 0 "L?" V 8240 4700 50  0000 C CNN
+F 0 "L1" V 8240 4700 50  0000 C CNN
 F 1 "33µH" V 8149 4700 50  0000 C CNN
 F 2 "" H 8050 4700 50  0001 C CNN
@@
 $EndComp
 $Comp
-L Device:CP_Small C?
+L Device:CP_Small C4
 U 1 1 60170C6A
 P 5800 4800
-F 0 "C?" H 5888 4846 50  0000 L CNN
+F 0 "C4" H 5888 4846 50  0000 L CNN
 F 1 "680µF" H 5888 4755 50  0000 L CNN
 F 2 "" H 5800 4800 50  0001 C CNN
@@
 Connection ~ 6800 5050
 $Comp
-L Device:CP_Small C?
+L Device:CP_Small C5
 U 1 1 6017D364
 P 8300 4800
-F 0 "C?" H 8388 4846 50  0000 L CNN
-F 1 "680µF" H 8388 4755 50  0000 L CNN
+F 0 "C5" H 8388 4846 50  0000 L CNN
+F 1 "220µF" H 8388 4755 50  0000 L CNN
 F 2 "" H 8300 4800 50  0001 C CNN
 F 3 "~" H 8300 4800 50  0001 C CNN
@@
 Connection ~ 8300 4700
 $Comp
-L power:+12V #PWR?
+L power:+12V #PWR06
 U 1 1 60185206
 P 8500 4700
-F 0 "#PWR?" H 8500 4550 50  0001 C CNN
+F 0 "#PWR06" H 8500 4550 50  0001 C CNN
 F 1 "+12V" V 8515 4828 50  0000 L CNN
 F 2 "" H 8500 4700 50  0001 C CNN
@@
 	8300 4700 8500 4700
 $Comp
-L Connector:Barrel_Jack_MountingPin J?
+L Connector:Barrel_Jack_MountingPin J2
 U 1 1 6018CC66
 P 5050 4700
-F 0 "J?" H 5107 5017 50  0000 C CNN
+F 0 "J2" H 5107 5017 50  0000 C CNN
 F 1 "Barrel_Jack_MountingPin" H 5107 4926 50  0000 C CNN
 F 2 "" H 5100 4660 50  0001 C CNN
@@
 	5350 5050 5800 5050
 Connection ~ 5800 5050
+Text Notes 5600 1750 0    100  ~ 0
+C2 and R1 values should/can be changed to\nincrease/decrease the duration of the spike period
 $EndSCHEMATC

Commit message: last implementation of the 6 spike and trigger board.
Parts:
- removed C1: 680pF, symbol pspice:CAP
- removed C2: 10µF, symbol pspice:CAP
- removed C3: 10nF, symbol pspice:CAP
- removed J1: Conn_Coaxial, symbol Connector:Conn_Coaxial
- removed Q1: MPSA42, Package_TO_SOT_THT:TO-92_Inline, symbol Transistor_BJT:MPSA42
- added C1, C14, C16, C2, C7, C8: 680pF, Capacitor_THT:C_Disc_D5.1mm_W3.2mm_P5.00mm, symbol Device:C_Small
- added C10, C17, C18, C3, C4, C9: 10nF, Capacitor_THT:C_Disc_D5.1mm_W3.2mm_P5.00mm, symbol Device:C_Small
- added C12, C13, C19, C20, C5, C6: 10µF, Capacitor_THT:C_Disc_D5.1mm_W3.2mm_P5.00mm, symbol Device:C_Small
- added D1, D10, D12, D18, D19, D2, D20, D21, D22, D23, D3, D4, D5, D6, D9: 1N4005, Diode_THT:D_DO-41_SOD81_P10.16mm_Horizontal, symbol Diode:1N4005
- added D15, D24, D25, D7, D8: 1N47xxA, Diode_THT:D_DO-41_SOD81_P10.16mm_Horizontal, symbol Diode:1N47xxA
- added J1: input_trigger_2, Connector_PinHeader_2.54mm:PinHeader_1x02_P2.54mm_Vertical, symbol Connector:Conn_01x02_Female
- added J10: input_trigger_6, Connector_PinHeader_2.54mm:PinHeader_1x02_P2.54mm_Vertical, symbol Connector:Conn_01x02_Female
- added J11: input_trigger_5, Connector_PinHeader_2.54mm:PinHeader_1x02_P2.54mm_Vertical, symbol Connector:Conn_01x02_Female
- added J12: to_solenoid_6, Connector_PinHeader_2.54mm:PinHeader_1x02_P2.54mm_Vertical, symbol Connector:Screw_Terminal_01x02
- added J13: to_solenoid_5, Connector_PinHeader_2.54mm:PinHeader_1x02_P2.54mm_Vertical, symbol Connector:Screw_Terminal_01x02
- added J2: input_trigger_1, Connector_PinHeader_2.54mm:PinHeader_1x02_P2.54mm_Vertical, symbol Connector:Conn_01x02_Female
- added J3: to_solenoid_2, Connector_PinHeader_2.54mm:PinHeader_1x02_P2.54mm_Vertical, symbol Connector:Screw_Terminal_01x02
- added J4: to_solenoid_1, Connector_PinHeader_2.54mm:PinHeader_1x02_P2.54mm_Vertical, symbol Connector:Screw_Terminal_01x02
- added J5: input_trigger_4, Connector_PinHeader_2.54mm:PinHeader_1x02_P2.54mm_Vertical, symbol Connector:Conn_01x02_Female
- added J6: input_trigger_3, Connector_PinHeader_2.54mm:PinHeader_1x02_P2.54mm_Vertical, symbol Connector:Conn_01x02_Female
- added J7: to_solenoid_4, Connector_PinHeader_2.54mm:PinHeader_1x02_P2.54mm_Vertical, symbol Connector:Screw_Terminal_01x02
- added Q1, Q17, Q18, Q2, Q9: MJH11021G, Package_TO_SOT_THT:TO-247-3_Vertical, symbol Device:Q_PNP_Darlington_BCE
- added Q11, Q12, Q13, Q19, Q20, Q21, Q22, Q3, Q4, Q5, Q6: MPSA42, Package_TO_SOT_THT:TO-92L_Inline_Wide, symbol dk_Transistors-Bipolar-BJT-Single:MPSA42
- added Q15, Q23, Q24, Q7, Q8: MJH11022G, Package_TO_SOT_THT:TO-247-3_Vertical, symbol Device:Q_NPN_Darlington_BCE
- added R1, R10, R15, R2, R22, R29, R30, R37, R38, R9: 10k, Resistor_THT:R_Axial_DIN0411_L9.9mm_D3.6mm_P12.70mm_Horizontal, symbol Device:R_Small
- added R11, R12, R19, R21, R25, R33, R34, R35, R36, R39, R40, R5, R6, R7, R8: 330, Resistor_THT:R_Axial_DIN0411_L9.9mm_D3.6mm_P12.70mm_Horizontal, symbol Device:R_Small
- added R13, R14, R27, R41, R42: 2k, Resistor_THT:R_Axial_DIN0411_L9.9mm_D3.6mm_P12.70mm_Horizontal, symbol Device:R_Small
- added R16, R3, R31, R32, R4: 4.7k, Resistor_THT:R_Axial_DIN0411_L9.9mm_D3.6mm_P12.70mm_Horizontal, symbol Device:R_Small
- added U1, U2, U3, U6, U7: LM555xM, Package_DIP:DIP-8_W7.62mm_LongPads, symbol Timer:LM555xM
- C11: renamed from C4; footprint (none) -> Capacitor_THT:CP_Radial_D10.0mm_P5.00mm
- C15: renamed from C5; footprint (none) -> Capacitor_THT:CP_Radial_D10.0mm_P5.00mm
- J8: renamed from J3; value to_solenoid -> to_solenoid_3; footprint (none) -> Connector_PinHeader_2.54mm:PinHeader_1x02_P2.54mm_Vertical
- J9: renamed from J2; footprint (none) -> digikey:Barrel_Jack_5.5mmODx2.1mmID_PJ-202A
- L1: footprint (none) -> Inductor_THT:L_Radial_D7.5mm_P3.50mm_Fastron_07P
- Q10: renamed from Q2; footprint (none) -> Package_TO_SOT_THT:TO-247-3_Vertical
- Q14: renamed from Q3; footprint digikey-footprints:TO-92-3 -> Package_TO_SOT_THT:TO-92L_Inline_Wide
- Q16: renamed from Q4; footprint (none) -> Package_TO_SOT_THT:TO-247-3_Vertical
- R17: renamed from R4; footprint (none) -> Resistor_THT:R_Axial_DIN0411_L9.9mm_D3.6mm_P12.70mm_Horizontal
- R18: renamed from R5; footprint (none) -> Resistor_THT:R_Axial_DIN0411_L9.9mm_D3.6mm_P12.70mm_Horizontal
- R20: renamed from R3; footprint (none) -> Resistor_THT:R_Axial_DIN0411_L9.9mm_D3.6mm_P12.70mm_Horizontal
- R23: renamed from R7; footprint (none) -> Resistor_THT:R_Axial_DIN0411_L9.9mm_D3.6mm_P12.70mm_Horizontal
- R24: renamed from R2; footprint (none) -> Resistor_THT:R_Axial_DIN0411_L9.9mm_D3.6mm_P12.70mm_Horizontal
- R26: renamed from R6; footprint (none) -> Resistor_THT:R_Axial_DIN0411_L9.9mm_D3.6mm_P12.70mm_Horizontal
- R28: renamed from R1; footprint (none) -> Resistor_THT:R_Axial_DIN0411_L9.9mm_D3.6mm_P12.70mm_Horizontal
- U4: renamed from U1; footprint Package_SO:SOIC-8_3.9x4.9mm_P1.27mm -> Package_DIP:DIP-8_W7.62mm_LongPads
- renumbered D3 to D11, D1 to D13, D4 to D14, D5 to D16, D2 to D17, U2 to U5
Connections:
- net +12V: now also R24.2, R28.2, U4.4 (R), U4.8 (VCC), D1.2 (A), D18.2 (A), D2.2 (A), D20.2 (A), D9.2 (A), R10.2, R13.2, R14.2, R22.2, R27.2, R37.2, R38.2, R41.2, R42.2, R9.2, U1.4 (R), U1.8 (VCC), U2.4 (R), U2.8 (VCC), U3.4 (R), U3.8 (VCC), U6.4 (R), U6.8 (VCC), U7.4 (R), U7.8 (VCC)
- net +24V: now also R17.1, Q1.2 (C), Q17.2 (C), Q18.2 (C), Q2.2 (C), Q9.2 (C), R1.1, R15.1, R2.1, R29.1, R30.1; no longer R17.2
- net GND: now also C10.1, C12.2, C13.2, C17.1, C18.1, C19.2, C20.2, C3.1, C4.1, C5.2, C6.2, C9.1, D10.2 (A), D19.2 (A), D21.2 (A), D3.2 (A), D4.2 (A), J1.2 (Pin_2), J10.2 (Pin_2), J11.2 (Pin_2), J2.2 (Pin_2), J5.2 (Pin_2), J6.2 (Pin_2), Q11.1 (E), Q12.1 (E), Q13.1 (E), Q15.3 (E), Q19.1 (E), Q20.1 (E), Q21.1 (E), Q22.1 (E), Q23.3 (E), Q24.3 (E), Q3.1 (E), Q4.1 (E), Q5.1 (E), Q6.1 (E), Q7.3 (E), Q8.3 (E), U1.1 (GND), U2.1 (GND), U3.1 (GND), U6.1 (GND), U7.1 (GND)
- net at R24.1, U4.2 (TR): now also Q12.3 (C)
- net at R23.1: now also Q14.2 (B); no longer U4.3 (Q)
- net at U4.5 (CV): now also C10.2
- net at U4.6 (THR), U4.7 (DIS): now also R28.1, C13.1; no longer R28.2
- net input_trigger3: now reaches R26.2
- net input_trigger3: now also C8.2, J6.1 (Pin_1)
- net at R20.2: now also C8.1
- net at D13.1 (K), R20.1: now also Q12.2 (B)
- net timed_trigger3: now reaches R23.2
- net timed_trigger3: now also U4.3 (Q); no longer Q14.2 (B)
- net at Q14.3 (C), R18.1: now also R17.2; no longer R17.1
- removed net VCC: R24.2, R28.1, U4.4 (R), U4.8 (VCC)
- new net: C20.1, R42.1, U7.6 (THR), U7.7 (DIS)
- new net: Q20.3 (C), R38.1, U7.2 (TR)
- new net: C18.2, U7.5 (CV)
- new net: C16.1, R34.2
- new net: D21.1 (K), Q20.2 (B), R34.1
- new net: Q22.2 (B), R36.1
- new net: Q22.3 (C), R30.2, R32.1
- new net: Q24.1 (B), R40.1
- new net: D20.1 (K), D23.1 (K), J13.1 (Pin_1), Q18.3 (E)
- new net: D25.1 (K), J13.2 (Pin_2), Q24.2 (C)
- new net: D23.2 (A), D25.2 (A)
- new net: Q18.1 (B), R32.2
- new net: C6.1, R14.1, U2.6 (THR), U2.7 (DIS)
- new net: Q4.3 (C), R10.1, U2.2 (TR)
- new net: C4.2, U2.5 (CV)
- new net: C2.1, R6.2
- new net: D4.1 (K), Q4.2 (B), R6.1
- new net: Q6.2 (B), R8.1
- new net: Q6.3 (C), R2.2, R4.1
- new net: Q8.1 (B), R12.1
- new net: D2.1 (K), D6.1 (K), J4.1 (Pin_1), Q2.3 (E)
- new net: D8.1 (K), J4.2 (Pin_2), Q8.2 (C)
- new net: D6.2 (A), D8.2 (A)
- new net: Q2.1 (B), R4.2
- new net: C19.1, R41.1, U6.6 (THR), U6.7 (DIS)
- new net: Q19.3 (C), R37.1, U6.2 (TR)
- new net: C17.2, U6.5 (CV)
- new net: C14.1, R33.2
- new net: D19.1 (K), Q19.2 (B), R33.1
- new net: Q21.2 (B), R35.1
- new net: Q21.3 (C), R29.2, R31.1
- new net: Q23.1 (B), R39.1
- new net: D18.1 (K), D22.1 (K), J12.1 (Pin_1), Q17.3 (E)
- new net: D24.1 (K), J12.2 (Pin_2), Q23.2 (C)
- new net: D22.2 (A), D24.2 (A)
- new net: Q17.1 (B), R31.2
- new net: D10.1 (K), Q11.2 (B), R19.1
- new net: Q11.3 (C), R22.1, U3.2 (TR)
- new net: D3.1 (K), Q3.2 (B), R5.1
- new net: Q3.3 (C), R9.1, U1.2 (TR)
- new net: C12.1, R27.1, U3.6 (THR), U3.7 (DIS)
- new net: C9.2, U3.5 (CV)
- new net: C7.1, R19.2
- new net: Q13.2 (B), R21.1
- new net: Q13.3 (C), R15.2, R16.1
- new net: Q15.1 (B), R25.1
- new net: D12.1 (K), D9.1 (K), J7.1 (Pin_1), Q9.3 (E)
- new net: D15.1 (K), J7.2 (Pin_2), Q15.2 (C)
- new net: D12.2 (A), D15.2 (A)
- new net: Q9.1 (B), R16.2
- new net: C5.1, R13.1, U1.6 (THR), U1.7 (DIS)
- new net: C3.2, U1.5 (CV)
- new net: C1.1, R5.2
- new net: Q5.2 (B), R7.1
- new net: Q5.3 (C), R1.2, R3.1
- new net: Q7.1 (B), R11.1
- new net: D1.1 (K), D5.1 (K), J3.1 (Pin_1), Q1.3 (E)
- new net: D7.1 (K), J3.2 (Pin_2), Q7.2 (C)
- new net: D5.2 (A), D7.2 (A)
- new net: Q1.1 (B), R3.2
- new net input_trigger1: C2.2, J2.1 (Pin_1), R12.2
- new net input_trigger2: C1.2, J1.1 (Pin_1), R11.2
- new net input_trigger4: C7.2, J5.1 (Pin_1), R25.2
- new net input_trigger5: C16.2, J11.1 (Pin_1), R40.2
- new net input_trigger6: C14.2, J10.1 (Pin_1), R39.2
- new net timed_trigger1: R8.2, U2.3 (Q)
- new net timed_trigger2: R7.2, U1.3 (Q)
- new net timed_trigger4: R21.2, U3.3 (Q)
- new net timed_trigger5: R36.2, U7.3 (Q)
- new net timed_trigger6: R35.2, U6.3 (Q)
- no-connect marks 0 -> 1
Other:
- note added: "C11 and R27\n values should/can be changed to\nincrease/decrease the duration of the spike period"
- note added: "C12 and R28 values should/can be changed to\nincrease/decrease the duration of the spike period"
- note added: "C19 and R41 values should/can be changed to\nincrease/decrease the duration of the spike period"
- note added: "C19 and R42 values should/can be changed to\nincrease/decrease the duration of the spike period"
- note added: "C5 and R13 values should/can be changed to\nincrease/decrease the duration of the spike period"
- note added: "C6 and R14 values should/can be changed to\nincrease/decrease the duration of the spike period"
- note removed: "C2 and R1 values should/can be changed to\nincrease/decrease the duration of the spike period"
- moved on the sheet: C11, C15, D11, D13, D14, D16, D17, J8, J9, L1, Q10, Q14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
